Commit message: added lucrezio with logical camera

File: urdf/lucrezio_with_logical.urdf.xacro (robot description, xacro)
@@ -7,5 +7,5 @@
   <xacro:property name="wheel_length" value="0.05" />
   <xacro:property name="wheel_radius" value="0.1" />
-  <xacro:property name="camera_link" value="0.05" />
+  <xacro:property name="camera_size" value="0.05" />
   <xacro:property name="camera_name" value="xtion" />
   <xacro:property name="M_PI" value="3.1415926535897931" />
@@ -194,11 +194,11 @@
       <origin xyz="0 0 0" rpy="0 0 0"/>
       <geometry>
-    <box size="${camera_link} ${camera_link} ${camera_link}"/>
-      </geometry>
-    </collision>
-    <visual>
-      <origin xyz="0 0 0" rpy="0 0 0"/>
-      <geometry>
-    <box size="${camera_link} ${camera_link} ${camera_link}"/>
+    <box size="${camera_size} ${camera_size} ${camera_size}"/>
+      </geometry>
+    </collision>
+    <visual>
+      <origin xyz="0 0 0" rpy="0 0 0"/>
+      <geometry>
+    <box size="${camera_size} ${camera_size} ${camera_size}"/>
       </geometry>
       <material name="red"/>
@@ -254,4 +254,47 @@
     </sensor>
   </gazebo>
+  <!-- LOGICAL CAMERA -->
+  <link name="logical_camera_link">
+    <collision>
+      <origin xyz="0 0 0" rpy="0 0 0"/>
+      <geometry>
+    <box size="${camera_size} ${camera_size} ${camera_size}"/>
+      </geometry>
+    </collision>
+    <visual>
+      <origin xyz="0 0 0" rpy="0 0 0"/>
+      <geometry>
+    <box size="${camera_size} ${camera_size} ${camera_size}"/>
+      </geometry>
+      <material name="red"/>
+    </visual>
+    <inertial>
+      <mass value="1e-5" />
+      <origin xyz="0 0 0" rpy="0 0 0"/>
+      <inertia ixx="1e-6" ixy="0" ixz="0" iyy="1e-6" iyz="0" izz="1e-6" />
+    </inertial>
+  </link>
+  <!-- LOGICAL CAMERA JOINT -->
+  <joint name="logical_camera_joint" type="fixed">
+    <axis xyz="0 1 0" />
+    <origin xyz="0 0 1.0" rpy="0 0 0"/>
+    <parent link="base_link"/>
+    <child link="logical_camera_link"/>
+  </joint>
+  <!-- LOGICAL CAMERA SENSOR -->
+  <gazebo reference="logical_camera_link">
+      <sensor name="logical_camera" type="logical_camera">
+        <plugin name="logical_camera_plugin" filename="liblogical_camera_plugin.so"/>
+          <logical_camera>
+            <near>0.02</near>
+            <far>5.0</far>
+            <horizontal_fov>${60.0*M_PI/180.0}</horizontal_fov>
+            <aspect_ratio>1.778</aspect_ratio>
+          </logical_camera>
+          <visualize>true</visualize>
+          <always_on>true</always_on>
+          <update_rate>10</update_rate>
+      </sensor>
+  </gazebo>
   <!-- Gazebo plugin for ROS Control -->
   <gazebo>

Commit message: boh

File: urdf/lucrezio_with_logical.urdf.xacro (robot description, xacro)
@@ -213,5 +213,5 @@
   <joint name="camera_joint" type="fixed">
     <axis xyz="0 1 0" />
-    <origin xyz="0 0 1.0" rpy="0 0 0"/>
+    <origin xyz="0 0 0.5" rpy="0 0 0"/>
     <parent link="base_link"/>
     <child link="camera_link"/>
