Commit message: now the resource paths are installation independent

File: urdf/lucrezio.urdf.xacro (robot description, xacro)
@@ -141,5 +141,5 @@
       <origin xyz="0 0 0" rpy="0 0 0" />
       <geometry>
-        <mesh filename="file:///home/dede/source/lucrezio/lucrezio_description/meshes/hokuyo.dae" />
+        <mesh filename="package://lucrezio_description/meshes/hokuyo.dae" />
       </geometry>
     </visual>

File: urdf/lucrezio_with_logical.urdf.xacro (robot description, xacro)
@@ -141,5 +141,5 @@
       <origin xyz="0 0 0" rpy="0 0 0" />
       <geometry>
-        <mesh filename="file:///home/dede/source/lucrezio/lucrezio_description/meshes/hokuyo.dae" />
+        <mesh filename="package://lucrezio_description/meshes/hokuyo.dae" />
       </geometry>
     </visual>
